File: Led-Controller.kicad_pcb (KiCad board)
At the start: 2 copper layers, 72.1 x 47.4 mm, 107 parts, among them J1 Program, J2 Barrel_Jack, J3 Screw_Terminal, J4 Screw_Terminal, J5 Ws2812 Conn, J6 Screw_Terminal, Q1 CSD18540Q5B, Q2 CSD18540Q5B, Q3 CSD18540Q5B, Q4 CSD18540Q5B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

Commit message: silk screen changes + review done
Routing:
- net GND: vias 133 -> 139
Other:
- outline, holes or cut-outs redrawn

Commit message: updated files according to FAb feedback and capabilities
Parts:
- moved C39 1.68 mm to (157.0, 102.2)
- moved C4 1.67 mm to (155.5, 100.4), turned to -90 degrees
- moved C3 1.31 mm to (152.8, 87.5), turned to -90 degrees
- moved C6 0.40 mm to (153.7, 92.5)
- moved R19 0.40 mm to (155.2, 92.5)
Routing:
- net Net-(U1-EN/SYNC): track 6.70 -> 10.8 mm
- net Net-(U2-PG): track 5.73 -> 9.79 mm
- net Net-(U1-PG): track 6.50 -> 10.4 mm
- net +9V: track 35.6 -> 38.4 mm
- net Net-(U2-EN/SYNC): track 8.04 -> 9.45 mm
- net +3.3V: track 59.7 -> 60.9 mm, vias 3 -> 4
- net GND: vias 139 -> 135
