File: Led-Controller.kicad_sch (KiCad schematic)
At the start: 107 parts, among them J1 Program, J2 Barrel_Jack, J3 Screw_Terminal, J4 Screw_Terminal, J5 Ws2812 Conn, J6 Screw_Terminal, Q1 CSD18540Q5B, Q2 CSD18540Q5B, Q3 CSD18540Q5B, Q4 CSD18540Q5B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

Commit message: Removed WS2812 Connector
Parts:
- removed C30: 0.1uf, Capacitor_SMD:C_0805_2012Metric, symbol Device:C_Small
- removed J4, J6: Screw_Terminal, TerminalBlock:TerminalBlock_bornier-2_P5.08mm, symbol Connector:Screw_Terminal_01x02
- removed J5: Ws2812 Conn, Connector_PinHeader_2.54mm:PinHeader_1x03_P2.54mm_Horizontal, symbol Connector_Generic:Conn_01x03
- removed JP1: Jumper_3_Open, Jumper:SolderJumper-3_P2.0mm_Open_TrianglePad1.0x1.5mm, symbol Jumper:Jumper_3_Open
- removed R33, R6: 90k, Resistor_SMD:R_0603_1608Metric, symbol Device:R_Small
- removed TP8: ~, TestPoint:TestPoint_Pad_D1.0mm, symbol Connector:TestPoint
- removed U9: SN74LV1T34DBV, Package_TO_SOT_SMD:SOT-23-5, symbol Logic_LevelTranslator:SN74LV1T34DBV
- added R32: 76.8k, Resistor_SMD:R_0603_1608Metric, symbol Device:R_Small
- TP1, TP2, TP3, TP4, TP5, TP6, TP7: value ~ -> (none)
Connections:
- net +9V: now also R32.1
- net at R7.1, U1.1 (FB): now also R32.2
- net DOUT: no longer names the net of U3.27 (IO16)
- no-connect marks 1 -> 0
Other:
- note removed: "Note : When using WS2812 the input supply should be 5V"
- note removed: "Output Stage WS2812"

Commit message: Did Producion changes
Parts:
- added H3, H4: MountingHole, MountingHole:MountingHole_3.2mm_M3_DIN965_Pad, symbol Mechanical:MountingHole
Other:
- note added: "VDD Min : 9V (if using RGBWWW) VDD Max : 30V"
- note removed: "VDD Min : 5V (if using WS2812) VDD Min : 9V (if using RGBWWW) VDD Max : 30V"
- moved on the sheet: C23, L3, R32, R7, TP2
